File: Schematics/LunettaAV_WIP.sch (EAGLE design)
At the start: 42 parts, among them IC1 4046N, IC2 4094N, IC3 TLC339P, IC4 7805T, IC5 4051N, IC6 4017N, IC7 4046N, U1 LM358

Commit message: scehmatics fixes
Parts:
- removed CLOCKDIV: (no value), adafruit:PINHD-1X6
- removed INH: 4040N, 40xx:4040N
- removed PLLCLOCK: (no value), jumper:JP1E
- removed TNSY5VIN: (no value), SparkFun-Retired:JUMPER-2PTH
- removed TNSYIN: (no value), jumper:JP4Q
- added D1, D2: 1N4148, diode:1N4148DO35-10
- added IC8: 4046N, 40xx:4046N
- added IC9: 40106N, 40xx:40106N
- added JP4: (no value), adafruit:PINHD-2X4
- added JP5: (no value), pinhead:PINHD-2X8
- added JP6: (no value), pinhead:PINHD-1X4
- added R18, R19, R20: 100K, MusicThingModular:RESISTOR7MM
- added R21: (no value), MusicThingModular:RESISTOR7MM
- added R22: 1K, MusicThingModular:RESISTOR7MM
- added VR3: 100K, MusicThingModular:9MM_SNAP-IN_POT_
- IC1: value 4046N -> TLC339P; device 40xx:4046N -> linear:TLC339P
- IC2: value 4094N -> 7805T; device 40xx:4094N -> linear:7805T
- IC3: value TLC339P -> 4046N; device linear:TLC339P -> 40xx:4046N
- IC4: value 7805T -> 4040N; device linear:7805T -> 40xx:4040N
- IC5: value 4051N -> 4017N; device 40xx:4051N -> 40xx:4017N
- IC6: value 4017N -> 4051N; device 40xx:4017N -> 40xx:4051N
- IC7: value 4046N -> 4094N; device 40xx:4046N -> 40xx:4094N
- JP1: device jumper:JP8Q -> adafruit:PINHD-2X4
- JP2: device jumper:JP5Q -> pinhead:PINHD-1X2
- JP3: device jumper:JP4E -> pinhead:PINHD-2X6
- R1, R2: value 4.7K -> 10K; device MusicThingModular:RESISTOR10MM_RESISTOR -> MusicThingModular:RESISTOR7MM
- R12: value 10K -> 100K
- R17: value 10K -> 1K
- R3: value 1K -> 10K; device MusicThingModular:RESISTOR10MM_RESISTOR -> MusicThingModular:RESISTOR7MM
- R5: value 10K -> 1K; device MusicThingModular:RESISTOR7MM -> MusicThingModular:RESISTOR10MM_RESISTOR
- R6, R9: value 10K -> 4.7K; device MusicThingModular:RESISTOR7MM -> MusicThingModular:RESISTOR10MM_RESISTOR
- renumbered ERASE to S3, OFFSET to S1, OLED1 to DISP$1, OLED2 to DISP$2, SCALER to VR2, SPEEDER to VR1, TEENSY to B1, WRITE to S2
Connections:
- removed net MINH: IC5A.INH, JP3.1, R14.1
- removed net PLL/64: CLOCKDIV.6, INHA.Q6
- new net DRONEOUT: R20.1, VR3.S
- new net GATEIN: JP6.4, R18.1
- new net MELODYBUFF: D1.C, VR3.E
- new net MIX: R19.2, R20.2, R21.2
- new net N$11: IC6A.INH, R13.2
- new net N$7: D1.A, D2.A, R18.2
- new net N$8: R22.2, S2.1
- new net VCAOUT: D2.C, R19.1
- net 3V3: now also R10.2, R11.2, R4.2, R9.2; no longer R1.2, R2.2, R5.2, R8.2
- net 5V: now also IC1A.-IN, IC1B.-IN, IC1C.-IN, IC1D.-IN, IC2.VO, JP2.1; no longer IC3A.-IN, IC3B.-IN, IC3C.-IN, IC3D.-IN, IC4.VO, TNSY5VIN.1
- net 9V: now also IC1P.V+, IC2.VI, IC3P.VDD, IC4P.VDD, IC6P.VCC, IC7A.OE, IC7A.STR, IC8P.VDD, R22.1; no longer IC1P.VDD, IC2A.STR, IC2P.VDD, IC3P.V+, IC4.VI, IC5P.VCC, INHP.VDD, S2.1
- net AUDIORATE: now also IC5A.CLK; no longer IC6A.CLK
- net BUFFCLOCK: now also IC7A.CLK; no longer IC2A.CLK
- net CLOCKSELECT: now also JP4.2, JP4.4, JP4.6, JP4.8; no longer JP2.1, JP2.3, JP2.5, JP2.7, JP2.9
- net DIN1: now also R5.2; no longer R3.2
- net GND: now also IC1P.V-, IC2.GND, IC3A.INH, IC3P.VSS, IC4P.VSS, IC6P.GND, IC6P.VEE, IC8P.VSS, R1.1, R13.1, R14.1, R15.1, R16.1, R2.1, R21.1, R5.1, R8.1, VR3.A; no longer IC1P.VSS, IC2P.VSS, IC3P.V-, IC4.GND, IC5P.GND, IC5P.VEE, IC7A.INH, INHP.VSS, R10.1, R11.1, R14.2, R15.2, R16.2, R17.2, R4.1, R9.1
- net MELODYOUT: now also IC5A.Q0; no longer IC6A.Q0
- net MOOX: now also IC6A.C, JP6.1, R16.2; no longer IC5A.C, JP3.4, R17.1
- net MOXO: now also IC6A.B, JP6.2, R15.2; no longer IC5A.B, JP3.3, R16.1
- net MXOO: now also IC6A.A, JP6.3, R14.2; no longer IC5A.A, JP3.2, R15.1
- net N$1: now also JP2.2; no longer TNSY5VIN.2
- net N$19: now also IC5A.RES, IC6A.X; no longer IC5A.X, IC6A.RES
- net N$2: now also IC3A.CX@2; no longer IC7A.CX@2
- net N$20: now also IC5A.Q2, IC6A.X0; no longer IC5A.X0, IC6A.Q2
- net N$21: now also IC5A.Q3, IC6A.X1; no longer IC5A.X1, IC6A.Q3
- net N$22: now also IC5A.Q4, IC6A.X2; no longer IC5A.X2, IC6A.Q4
- net N$23: now also IC5A.Q5, IC6A.X3; no longer IC5A.X3, IC6A.Q5
- net N$24: now also IC5A.Q6, IC6A.X4; no longer IC5A.X4, IC6A.Q6
- net N$25: now also IC5A.Q7, IC6A.X5; no longer IC5A.X5, IC6A.Q7
- net N$26: now also IC5A.Q8, IC6A.X6; no longer IC5A.X6, IC6A.Q8
- net N$27: now also IC5A.Q9, IC6A.X7; no longer IC5A.X7, IC6A.Q9
- net N$28: now also IC7A.D, R17.1; no longer IC2A.D, R13.1
- net N$3: now also R6.1; no longer R1.1
- net N$4: now also R9.1; no longer R2.1
- net N$5: now also IC3A.CX@1; no longer IC7A.CX@1
- net N$6: now also IC3A.R1, R12.2; no longer IC7A.R1, R4.2
- net OOX: now also IC1D.+IN, JP1.1, JP1.2, R8.2; no longer IC3D.+IN, R12.2, TNSYIN.1, TNSYIN.2
- net OXO: now also IC1C.+IN, JP1.3, JP1.4, R3.2; no longer IC3C.+IN, R11.2, TNSYIN.3, TNSYIN.4
- net PLL/16: now also IC4A.Q4, JP3.10, JP3.9; no longer CLOCKDIV.4, INHA.Q4, JP2.2
- net PLL/2: now also IC4A.Q1, JP3.3, JP3.4, JP4.3; no longer CLOCKDIV.1, INHA.Q1, JP2.8
- net PLL/32: now also IC4A.Q5, JP3.11, JP3.12; no longer CLOCKDIV.5, INHA.Q5
- net PLL/4: now also IC4A.Q2, JP3.5, JP3.6, JP4.5; no longer CLOCKDIV.2, INHA.Q2, JP2.6
- net PLL/8: now also IC4A.Q3, JP3.7, JP3.8, JP4.7; no longer CLOCKDIV.3, INHA.Q3, JP2.4
- net PLLCLOCKOUT: now also IC3A.VCOOUT, IC4A.P1, JP3.1, JP3.2, JP4.1; no longer IC7A.VCOOUT, INHA.P1, JP2.10, PLLCLOCK.1, PLLCLOCK.2
- net RESET: now also IC1A.+IN, JP1.7, JP1.8, R1.2; no longer IC3A.+IN, R9.2, TNSYIN.7, TNSYIN.8
- net SPEEDYBUFF: now also IC3A.VCOIN; no longer IC7A.VCOIN
- net SR1: now also IC7A.Q1, JP5.1, JP5.2; no longer IC2A.Q1, JP1.1, JP1.2
- net SR2: now also IC7A.Q2, JP5.3, JP5.4; no longer IC2A.Q2, JP1.3, JP1.4
- net SR3: now also IC7A.Q3, JP5.5, JP5.6; no longer IC2A.Q3, JP1.5, JP1.6
- net SR4: now also IC7A.Q4, JP5.7, JP5.8; no longer IC2A.Q4, JP1.7, JP1.8
- net SR5: now also IC7A.Q5, JP5.10, JP5.9; no longer IC2A.Q5, JP1.10, JP1.9
- net SR6: now also IC7A.Q6, JP5.11, JP5.12; no longer IC2A.Q6, JP1.11, JP1.12
- net SR7: now also IC7A.Q7, JP5.13, JP5.14; no longer IC2A.Q7, JP1.13, JP1.14
- net SR8: now also IC7A.Q8, JP5.15, JP5.16, R17.2; no longer IC2A.Q8, JP1.15, JP1.16, R13.2
- net TNSYOOX: now also IC1D.OUT, R11.1; no longer IC3D.OUT, R8.1
- net TNSYOXO: now also IC1C.OUT, R10.1; no longer IC3C.OUT, R7.1
- net TNSYRES: now also IC1A.OUT, R4.1; no longer IC3A.OUT, R5.1
- net TNSYXOO: now also IC1B.OUT, R7.1; no longer IC3B.OUT, R6.1
- net XOO: now also IC1B.+IN, JP1.5, JP1.6, R2.2; no longer IC3B.+IN, R10.2, TNSYIN.5, TNSYIN.6
