File: Schematics/LunettaAV_WIP.brd (EAGLE design)
At the start: 160 x 100 mm, 99 parts, among them IC1 7809\, IC10 4051N, IC2 7805, IC3 4040N, IC4 TLC339P, IC5 4046N, IC6 4094N, IC7 40106N, IC8 4046N, IC9 4017N, J1 POWER_JACKPOWER_JACK_SLOT, J3 WQP-PJ301M-12_JACK, U1 LM358, U2 LM358, U3 MICROCHIP_MCP41050-I-PMICROCH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

Commit message: brd init
Parts:
- removed CLOCK-OUT, J3: WQP-PJ301M-12_JACK, MusicThingModular:WQP-PJ301M-12_JACK
- removed FDBCK: (no value), MusicThingModular:9MM_SNAP-IN_POT
- removed J2: (no value), SparkFun-Connectors:1X04_LONGPADS
- removed PITCH: 100K, MusicThingModular:9MM_SNAP-IN_POT
- removed S1, S2, S3: MOMENTARY-SWITCH-SPST-PTH-12MM, SparkFun-Switches:TACTILE_SWITCH_PTH_12MM
- removed VR1: (no value), MusicThingModular:BOURNS_3362P_TRIMMER
- added CLOCKOUT, OUTPUT: WQP-PJ301M-12_JACK, MusicThingModular:WQP-PJ301M-12_JACK
- added ERASE, PATTERNOFFSET, WRITE: MOMENTARY-SWITCH-SPST-PTH-12MM, SparkFun-Switches:TACTILE_SWITCH_PTH_12MM
- added FDBK: 100k, MusicThingModular:9MM_SNAP-IN_POT
- added FREQ: 100K, MusicThingModular:9MM_SNAP-IN_POT
- added JP6: (no value), pinhead:2X08
- added VR4: (no value), MusicThingModular:BOURNS_3362P_TRIMMER
- C10, C15, C26, C7, C9: value 0.1uF -> 10uF; device SparkFun-Capacitors:CAP-PTH-SMALL-KIT -> SparkFun-Capacitors:CPOL-RADIAL-2.5MM-5MM
- C14: value .1uF -> 0.1uF; device capacitor-wima:C2.5-2 -> SparkFun-Capacitors:CAP-PTH-SMALL-KIT
- C18: value 47uF -> 0.1uF; device SparkFun-Capacitors:CPOL-RADIAL-2.5MM-5MM -> SparkFun-Capacitors:CAP-PTH-SMALL-KIT
- C19: value 0.1uF -> .1uF; device SparkFun-Capacitors:CAP-PTH-SMALL-KIT -> capacitor-wima:C2.5-2
- C2, C24, C25, C3, C5: value 10uF -> 0.1uF; device SparkFun-Capacitors:CPOL-RADIAL-2.5MM-5MM -> SparkFun-Capacitors:CAP-PTH-SMALL-KIT
- C20: value 0.1uF -> 47uF; device SparkFun-Capacitors:CAP-PTH-SMALL-KIT -> SparkFun-Capacitors:CPOL-RADIAL-2.5MM-5MM
- IC1: value 7809\ -> TLC339P; device v-reg:78XXS -> linear:DIL14
- IC10: value 4051N -> 40106N; device 40xx:DIL16 -> 40xx:DIL14
- IC2: value 7805 -> 4046N; device v-reg:78XXS -> 40xx:DIL16
- IC3: value 4040N -> 7809\; device 40xx:DIL16 -> v-reg:78XXS
- IC4: value TLC339P -> 4040N; device linear:DIL14 -> 40xx:DIL16
- IC5: value 4046N -> 7805; device 40xx:DIL16 -> v-reg:78XXS
- IC6: value 4094N -> 4017N
- IC7: value 40106N -> 4051N; device 40xx:DIL14 -> 40xx:DIL16
- IC8: value 4046N -> 4094N
- IC9: value 4017N -> 4046N
- JP1: device pinhead:1X02 -> jumper:JP4
- JP2: device adafruit:2X04 -> pinhead:1X02
- JP4: device pinhead:2X08 -> adafruit:2X04
- MIX: value (none) -> 100k
- R1, R2: value 4.7K -> 10K
- R10: value 10K -> 4.7k
- R12: value 100K -> 4.7k
- R13, R3: value 1K -> 10K
- R14: value 1K -> 4.7k
- R15: value LDR -> 100K; device rcl:0204V -> MusicThingModular:7MM_RESISTOR
- R17, R29: value 10k -> 100k
- R18: value 10K -> 10k
- R19, R20: value 10K -> 100k
- R21: value 2.2k -> 10k
- R22: value 100k -> 1K
- R23: value 100k -> 10K
- R24, R25: value 4.7k -> 10K
- R26: value 4.7k -> 1K
- R28: value 100k -> LDR; device MusicThingModular:7MM_RESISTOR -> rcl:0204V
- R30: value 100k -> 2.2k
- R5, R9: value 10K -> 4.7K
- R6: value 10K -> 1K
- U2: value LM358 -> MICROCHIP_MCP41050-I-PMICROCHIP_MCP41050-I-P_0_0; device SparkFun-IC-Amplifiers:DIP08 -> MCP41050:MICROCHIP_MCP41050-I-P_0
- U3: value MICROCHIP_MCP41050-I-PMICROCHIP_MCP41050-I-P_0_0 -> LM358; device MCP41050:MICROCHIP_MCP41050-I-P_0 -> SparkFun-IC-Amplifiers:DIP08
- moved R14 206.0 mm to (92.7, 76.2)
- moved C26 195.3 mm to (90.2, 59.7)
- moved U2 186.9 mm to (94.0, 92.7), turned to 90 degrees
- moved R4 186.8 mm to (81.3, 118.1)
- moved R12 185.3 mm to (92.7, 80.0)
- moved R13 180.6 mm to (81.3, 106.7)
- moved D1 172.5 mm to (68.6, 132.1), turned to 180 degrees
- moved R22 169.6 mm to (52.1, 12.7)
- moved IC10 167.7 mm to (74.9, 71.1)
- moved R10 164.6 mm to (92.7, 83.8)
- moved R11 160.1 mm to (81.3, 110.5)
- moved B1 155.3 mm to (97.8, 118.1), turned to 180 degrees
- moved R26 136.1 mm to (52.1, 7.62)
- moved IC5 129.2 mm to (29.2, 124.5)
- moved OL96$1 125.3 mm to (77.5, 38.1)
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Connections:
- net 3V3: now also C2.1, C3.1, PATTERNOFFSET.1, R11.2, R13.2, R9.2; no longer C1.1, C4.1, R1.2, R2.2, R6.2, S1.1
- net 5V: now also C10.1, C15.1, C16.1, IC1.10, IC1.4, IC1.6, IC1.8, IC5.OUT, JP2.1, R10.2, R12.2, R14.2, U2.8; no longer C25.1, C26.1, C5.1, IC2.OUT, IC4.10, IC4.4, IC4.6, IC4.8, JP1.1, R24.2, R25.2, R26.2, U3.8
- net 9V: now also C1.1, C14.1, C18.1, C4.1, C5.1, IC1.3, IC10.14, IC2.16, IC3.OUT, IC4.16, IC5.IN, IC7.16, IC8.1, IC8.15, R22.1, U3.8; no longer C15.1, C16.1, C3.1, C6.1, C7.1, IC1.OUT, IC10.16, IC2.IN, IC3.16, IC4.3, IC5.16, IC6.1, IC6.15, IC7.14, R13.1, U2.8
- net AUDIORATE: now also IC10.6, IC6.14; no longer IC7.6, IC9.14
- net BOUNCEPIN: now also PATTERNOFFSET.3, R6.2; no longer R3.2, S1.3
- net BUFFCLOCK: now also IC8.3, R16.1; no longer IC6.3, R22.1
- net BUFFMEL: now also R31.1, U3.6, U3.7; no longer R16.1, U2.6, U2.7
- net CLOCKSELECT: now also JP4.2, JP4.4, JP4.6, JP4.8; no longer JP2.2, JP2.4, JP2.6, JP2.8
- net DCIN: now also C7.1, IC3.IN; no longer C2.1, IC1.IN
- net DPOTDATA: now also R12.1, U2.3; no longer R25.1, U3.3
- net DPOTSCK: now also R14.1, U2.2; no longer R26.1, U3.2
- net DPOTSEL: now also R10.1, U2.1; no longer R24.1, U3.1
- net GND: now also C10.2, C19.2, C20.2, C21.2, C22.1, C24.1, CLOCKOUT.P$3_SLEEVE, ERASE.1, FDBK.1, IC1.12, IC10.11, IC10.13, IC10.9, IC2.5, IC2.8, IC3.GND, IC4.8, IC5.GND, IC6.13, IC7.6, IC7.8, J1.GNDBREAK, OUTPUT.P$3_SLEEVE, R1.1, R15.1, R17.1, R2.1, R23.1, R24.1, R25.1, R29.2, R6.1, U2.5, U2.6, VR4.3; no longer C19.1, C20.1, C22.2, C25.2, C26.2, C6.2, CLOCK-OUT.P$3_SLEEVE, FDBCK.1, IC1.GND, IC10.6, IC10.8, IC2.GND, IC3.8, IC4.12, IC5.5, IC5.8, IC7.11, IC7.13, IC7.9, IC9.13, J3.P$3_SLEEVE, R10.1, R11.1, R12.1, R18.1, R19.1, R23.2, R28.1, R31.1, R9.1, S3.1, U3.5, U3.6, VR1.3
- net LDRIVER: now also R19.1; no longer R30.1
- net MELODYOUT: now also IC6.3, U3.5; no longer IC9.3, U2.5
- net MOOX: now also IC7.9, R25.2; no longer IC10.9, R20.2
- net MOXO: now also IC7.10, R24.2; no longer IC10.10, R19.2
- net MXOO: now also IC7.11, R23.2; no longer IC10.11, R18.2
- net N$1: now also JP2.2; no longer JP1.2
- net N$10: now also IC10.4, IC10.5; no longer IC7.4, IC7.5
- net N$11: now also C19.1, FREQ.2, IC10.1, R28.2; no longer C14.1, IC7.1, PITCH.2, R15.2
- net N$12: now also C25.1; no longer C21.1
- net N$13: now also R27.2, R29.1, U3.3; no longer R22.2, R23.1, U2.3
- net N$14: now also U3.1, U3.2; no longer U2.1, U2.2
- net N$15: now also R30.2; no longer R21.2
- net N$16: now also C20.1; no longer C18.1
- net N$17: now also C22.2; no longer C20.2
- net N$18: now also C21.1; no longer C22.1
- net N$19: now also IC6.15, IC7.3; no longer IC10.3, IC9.15
- net N$2: now also C6.2, IC2.7; no longer C10.2, IC5.7
- net N$20: now also IC6.4, IC7.13; no longer IC10.13, IC9.4
- net N$21: now also IC6.7, IC7.14; no longer IC10.14, IC9.7
- net N$22: now also IC6.10, IC7.15; no longer IC10.15, IC9.10
- net N$23: now also IC6.1, IC7.12; no longer IC10.12, IC9.1
- net N$24: now also IC6.5, IC7.1; no longer IC10.1, IC9.5
- net N$25: now also IC6.6, IC7.5; no longer IC10.5, IC9.6
- net N$26: now also IC6.9, IC7.2; no longer IC10.2, IC9.9
- net N$27: now also IC6.11, IC7.4; no longer IC10.4, IC9.11
- net N$28: now also ERASE.3, IC8.2, R26.1, WRITE.3; no longer IC6.2, R14.1, S2.3, S3.3
- net N$29: now also R31.2, R32.1; no longer R16.2, R17.1
- net N$3: now also R5.1; no longer R1.1
- net N$30: now also FDBK.2, R32.2; no longer FDBCK.2, R17.2
- net N$31: now also C24.2; no longer C19.2
- net N$32: now also CLOCKOUT.P$1_TIP; no longer CLOCK-OUT.P$1_TIP
- net N$33: now also R30.1, U2.7; no longer R21.1, U3.7
- net N$34: now also R16.2, R17.2; no longer R27.2, R28.2
- net N$35: now also R18.1; no longer R29.1
- net N$36: now also R18.2; no longer R29.2
- net N$37: now also R19.2, R20.2; no longer R30.2, R31.2
- net N$38: now also R21.1; no longer R32.1
- net N$39: now also R21.2; no longer R32.2
- net N$4: now also R9.1; no longer R2.1
- net N$40: now also OUTPUT.P$1_TIP, VR4.2; no longer J3.P$1_TIP, VR1.2
- net N$41: now also C26.2, VR4.1; no longer C24.2, VR1.1
- net N$5: now also C6.1, IC2.6; no longer C10.1, IC5.6
- net N$6: now also IC2.11, R15.2; no longer IC5.11, R12.2
- net N$7: now also C25.2; no longer C21.2
- net N$8: now also R22.2, WRITE.1; no longer R13.2, S2.1
- net N$9: now also FREQ.3, IC10.2, IC10.3, R28.1; no longer IC7.2, IC7.3, PITCH.3, R15.1
- net OOX: now also IC1.11, JP1.4, R8.2; no longer IC4.11, J2.4, R11.2
- net OUT: now also C26.1; no longer C24.1
- net OXO: now also IC1.9, JP1.3, R3.2; no longer IC4.9, J2.3, R10.2
- net PLL/16: now also IC4.5; no longer IC3.5
- net PLL/2: now also IC4.9, JP4.3; no longer IC3.9, JP2.3
- net PLL/32: now also IC4.3; no longer IC3.3
- net PLL/4: now also IC4.7, JP4.5; no longer IC3.7, JP2.5
- net PLL/8: now also IC4.6, JP4.7; no longer IC3.6, JP2.7
- net PLLCLOCKOUT: now also IC2.4, IC4.10, JP4.1; no longer IC3.10, IC5.4, JP2.1
- net RESET: now also IC1.5, JP1.1, R1.2; no longer IC4.5, J2.1, R8.2
- net SPEEDYBUFF: now also IC2.9; no longer IC5.9
- net SR1: now also IC8.4, JP6.1, JP6.2; no longer IC6.4, JP4.1, JP4.2
- net SR2: now also IC8.5, JP6.3, JP6.4; no longer IC6.5, JP4.3, JP4.4
- net SR3: now also IC8.6, JP6.5, JP6.6; no longer IC6.6, JP4.5, JP4.6
- net SR4: now also IC8.7, JP6.7, JP6.8; no longer IC6.7, JP4.7, JP4.8
- net SR5: now also IC8.14, JP6.10, JP6.9; no longer IC6.14, JP4.10, JP4.9
- net SR6: now also IC8.13, JP6.11, JP6.12; no longer IC6.13, JP4.11, JP4.12
- net SR7: now also IC8.12, JP6.13, JP6.14; no longer IC6.12, JP4.13, JP4.14
- net SR8: now also IC8.11, JP6.15, JP6.16, R26.2; no longer IC6.11, JP4.15, JP4.16, R14.2
- net TNSYOOX: now also IC1.13, R13.1; no longer IC4.13, R7.1
- net TNSYOXO: now also IC1.14, R11.1; no longer IC4.14, R6.1
- net TNSYRES: now also IC1.2; no longer IC4.2
- net TNSYXOO: now also IC1.1, R7.1; no longer IC4.1, R5.1
- net XOO: now also IC1.7, JP1.2, R2.2; no longer IC4.7, J2.2, R9.2
Other:
- board size 160 x 100 mm -> 7 x 7 mm

Commit message: PCB Design
Parts:
- removed DD1: PT2399, ic-princeton-technologies:DIP-16
- removed IC9: 4046N, 40xx:DIL16
- removed JP1, JP5: (no value), jumper:JP4
- removed JP2: (no value), pinhead:1X02
- removed JP3: (no value), pinhead:2X06
- removed JP6: (no value), pinhead:2X08
- removed LED1, LED2: (no value), led:LED3MM
- removed U2: MICROCHIP_MCP41050-I-PMICROCHIP_MCP41050-I-P_0_0, MCP41050:MICROCHIP_MCP41050-I-P_0
- added CLOCK, MS4: (no value), SparkFun-LED:LED_3MM
- added CLOCKDIV: (no value), pinhead:2X06
- added MCP41050: MICROCHIP_MCP41050-I-PMICROCHIP_MCP41050-I-P_0_0, MCP41050:MICROCHIP_MCP41050-I-P_0
- added MUXSELECT, TNSYSELECT: (no value), jumper:JP4
- added PT2399: PT2399, ic-princeton-technologies:DIP-16
- added SHIFTREG: (no value), pinhead:2X08
- added TNSYPWR: (no value), pinhead:1X02
- C14: value 0.1uF -> 10uF; device SparkFun-Capacitors:CAP-PTH-SMALL-KIT -> SparkFun-Capacitors:CPOL-RADIAL-2.5MM-5MM
- ERASE, PATTERNOFFSET, WRITE: value MOMENTARY-SWITCH-SPST-PTH-12MM -> (none)
- J1: value POWER_JACKPOWER_JACK_SLOT -> (none)
- moved C21 211.6 mm to (97.8, 24.1)
- moved C22 209.3 mm to (108.0, 24.1)
- moved R21 204.3 mm to (120.7, 80.0)
- moved C8 204.0 mm to (73.7, 39.4)
- moved C25 199.6 mm to (102.9, 48.3)
- moved C16 196.5 mm to (82.5, 39.4)
- moved R8 194.4 mm to (109.2, 67.3)
- moved R20 192.8 mm to (120.7, 87.6)
- moved R30 189.2 mm to (97.8, 30.5)
- moved R3 182.7 mm to (109.2, 74.9)
- moved R19 181.4 mm to (120.7, 95.2)
- moved C24 180.0 mm to (94.0, 48.3)
- moved C19 172.0 mm to (87.6, 55.9), turned to 90 degrees
- moved R2 171.1 mm to (109.2, 82.5)
- moved C3 166.9 mm to (47.0, 24.1)
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Connections:
- removed net 3V: B1.3V
- net 3V3: now also B1.3V, C14.1
- net 5V: now also MCP41050.8, PT2399.1, TNSYPWR.1; no longer DD1.1, JP2.1, U2.8
- net 9V: now also CLOCK.A, MS4.A; no longer C14.1, IC9.16, LED1.A, LED2.A
- net DPOTDATA: now also MCP41050.3; no longer U2.3
- net DPOTSCK: now also MCP41050.2; no longer U2.2
- net DPOTSEL: now also MCP41050.1; no longer U2.1
- net GND: now also MCP41050.4, MCP41050.5, MCP41050.6, PT2399.12, PT2399.3, PT2399.4; no longer DD1.12, DD1.3, DD1.4, IC9.8, U2.4, U2.5, U2.6
- net LDRIVER: now also MUXSELECT.4; no longer JP5.4
- net MOOX: now also MUXSELECT.3; no longer JP5.3
- net MOXO: now also MUXSELECT.2; no longer JP5.2
- net MXOO: now also MUXSELECT.1; no longer JP5.1
- net N$1: now also TNSYPWR.2; no longer JP2.2
- net N$12: now also PT2399.10; no longer DD1.10
- net N$15: now also PT2399.6; no longer DD1.6
- net N$16: now also PT2399.2; no longer DD1.2
- net N$17: now also PT2399.7; no longer DD1.7
- net N$18: now also PT2399.8; no longer DD1.8
- net N$29: now also PT2399.16; no longer DD1.16
- net N$30: now also PT2399.15; no longer DD1.15
- net N$31: now also PT2399.11; no longer DD1.11
- net N$33: now also MCP41050.7; no longer U2.7
- net N$36: now also CLOCK.K; no longer LED1.K
- net N$39: now also MS4.K; no longer LED2.K
- net N$7: now also PT2399.9; no longer DD1.9
- net OOX: now also TNSYSELECT.4; no longer JP1.4
- net OXO: now also TNSYSELECT.3; no longer JP1.3
- net PLL/16: now also CLOCKDIV.10, CLOCKDIV.9; no longer JP3.10, JP3.9
- net PLL/2: now also CLOCKDIV.3, CLOCKDIV.4; no longer JP3.3, JP3.4
- net PLL/32: now also CLOCKDIV.11, CLOCKDIV.12; no longer JP3.11, JP3.12
- net PLL/4: now also CLOCKDIV.5, CLOCKDIV.6; no longer JP3.5, JP3.6
- net PLL/8: now also CLOCKDIV.7, CLOCKDIV.8; no longer JP3.7, JP3.8
- net PLLCLOCKOUT: now also CLOCKDIV.1, CLOCKDIV.2; no longer JP3.1, JP3.2
- net RESET: now also TNSYSELECT.1; no longer JP1.1
- net SR1: now also SHIFTREG.1, SHIFTREG.2; no longer JP6.1, JP6.2
- net SR2: now also SHIFTREG.3, SHIFTREG.4; no longer JP6.3, JP6.4
- net SR3: now also SHIFTREG.5, SHIFTREG.6; no longer JP6.5, JP6.6
- net SR4: now also SHIFTREG.7, SHIFTREG.8; no longer JP6.7, JP6.8
- net SR5: now also SHIFTREG.10, SHIFTREG.9; no longer JP6.10, JP6.9
- net SR6: now also SHIFTREG.11, SHIFTREG.12; no longer JP6.11, JP6.12
- net SR7: now also SHIFTREG.13, SHIFTREG.14; no longer JP6.13, JP6.14
- net SR8: now also SHIFTREG.15, SHIFTREG.16; no longer JP6.15, JP6.16
- net XOO: now also TNSYSELECT.2; no longer JP1.2
Routing:
- net GND: track 0.00 -> 856.1 mm, vias 0 -> 1
- net 9V: track 0.00 -> 367.0 mm, vias 0 -> 2
- net 3V3: track 0.00 -> 304.5 mm, vias 0 -> 8
- net SPEEDPIN: track 0.00 -> 265.4 mm, vias 0 -> 2
- net N$28: track 0.00 -> 262.5 mm, vias 0 -> 3
- net 5V: track 0.00 -> 234.7 mm, vias 0 -> 1
- net XOO: track 0.00 -> 233.9 mm, vias 0 -> 3
- net OXO: track 0.00 -> 224.9 mm, vias 0 -> 3
- net BUFFMEL: track 0.00 -> 224.0 mm, vias 0 -> 2
- net OOX: track 0.00 -> 215.2 mm, vias 0 -> 2
- net N$8: track 0.00 -> 197.5 mm, vias 0 -> 2
- net DENSITYPIN: track 0.00 -> 195.7 mm, vias 0 -> 4
- net RESET: track 0.00 -> 189.0 mm, vias 0 -> 3
- net LDRIVER: track 0.00 -> 171.0 mm, vias 0 -> 5
- net BOUNCEPIN: track 0.00 -> 167.4 mm, vias 0 -> 5
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- added copper zone on layer 1, net GND
- added copper zone on layer 16, net GND
Other:
- board size 7 x 7 mm -> 128.3 x 138.4 mm
- board text added: "CLOCK OUT"
- board text added: "CLOCK SELECT"
- board text added: "DENSITY"
- board text added: "ERASE"
- board text added: "FDBK"
- board text added: "FREQ"
- board text added: "INPUTS"
- board text added: "MIX"
- board text added: "N8IR"
- board text added: "OUT"
- board text added: "OUTPUTS"
- board text added: "PATTERN"
- board text added: "SPEED"
- board text added: "Sourya Sen 2023"
- board text added: "WRITE"
- board text added: "experimental audiovisual synthesiser and phrase generator"

Commit message: redo routing
Parts:
- moved R22 87.3 mm to (97.8, 22.9)
- moved ERASE 34.3 mm to (120.7, 14.0)
- moved WRITE 34.3 mm to (102.9, 14.0)
- moved FDBK 34.3 mm to (68.6, 12.7)
- moved MIX 34.3 mm to (85.1, 12.7)
- moved C21 27.9 mm to (111.8, 48.3)
- moved C22 2.54 mm to (108.0, 26.7)
- moved R11 1.27 mm to (97.8, 123.2)
- moved R13 1.27 mm to (96.5, 116.8)
- moved R4 1.27 mm to (97.8, 133.3)
- moved R7 1.27 mm to (97.8, 128.3)
Connections:
- net N$3 renamed SCL
- net N$4 renamed SDA
Routing:
- net N$8: track 197.5 -> 14.5 mm, vias 2 -> 0
- net N$37: track 143.3 -> 267.3 mm, vias 2 -> 4
- net MXOO: track 157.2 -> 265.6 mm, vias 3 -> 4
- net DENSITYPIN: track 195.7 -> 297.5 mm
- net BOUNCEPIN: track 167.4 -> 259.9 mm, vias 5 -> 4
- net GND: track 856.1 -> 932.6 mm, vias 1 -> 2
- net N$28: track 262.5 -> 186.9 mm, vias 3 -> 8
- net RESET: track 189.0 -> 260.1 mm
- net SPEEDPIN: track 265.4 -> 332.7 mm, vias 2 -> 5
- net 9V: track 367.0 -> 420.5 mm, vias 2 -> 5
- net PLL/4: track 51.0 -> 104.3 mm, vias 0 -> 3
- net BUFFMEL: track 224.0 -> 173.8 mm, vias 2 -> 4
- net PLL/16: track 71.2 -> 108.2 mm, vias 2 -> 4
- net N$33: track 34.1 -> 70.7 mm
- net N$11: track 108.7 -> 134.5 mm, vias 1 -> 3
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Other:
- board size 128.3 x 138.4 mm -> 129.5 x 138.4 mm
- board text added: "By pressing down a special key It plays a little melody"
- board text added: "N8IR experimental audiovisual synthesiser and phrase generator designed by sourya sen board version 1.0"
- board text added: "this project wouldn't be possible without the knowledge shared on electro-music forums and previous work by andy murkin"

Commit message: fix minor schematic issues for a cleaner bom
Parts:
- 7809: value 7809\ -> 7809
- C19: value .1uF -> 1uF; device capacitor-wima:C2.5-2 -> capacitor-wima:C5B3.5
- DENSITY, FREQ, R15, SPEED: value 100K -> 100k
- MCP41050: value MICROCHIP_MCP41050-I-PMICROCHIP_MCP41050-I-P_0_0 -> MCP41050
- R1, R11, R13, R2, R23, R24, R25, R3, R4, R7, R8: value 10K -> 10k
- R22, R26, R6: value 1K -> 1k
- R5, R9: value 4.7K -> 4.7k
- moved C26 6.84 mm to (109.2, 61.0)
- moved C24 5.68 mm to (91.4, 53.3), turned to 90 degrees
- moved C21 5.08 mm to (106.7, 48.3)
- moved C25 5.08 mm to (97.8, 48.3)
- moved C20 4.02 mm to (82.5, 45.7)
- moved VR4 3.81 mm to (120.7, 68.6), turned to 0 degrees
- moved C19 2.54 mm to (85.1, 55.9)
- renumbered IC10 to 40106, IC2 to 4046, IC3 to 7809, IC4 to 4040, IC5 to 7805, IC6 to 4017, IC7 to 4051, IC8 to 4094, U1 to LM358-1, U3 to LM358-2
Routing:
- net MXOO: track 265.6 -> 139.8 mm, vias 4 -> 2
- net N$37: track 267.3 -> 144.5 mm, vias 4 -> 1
- net N$28: track 186.9 -> 251.9 mm, vias 8 -> 2
- net RESET: track 260.1 -> 196.5 mm, vias 3 -> 5
- net PLL/16: track 108.2 -> 46.1 mm, vias 4 -> 2
- net SR7: track 115.4 -> 68.7 mm
- net BUFFMEL: track 173.8 -> 220.3 mm, vias 4 -> 3
- net LDRIVER: track 160.3 -> 205.4 mm, vias 1 -> 3
- net N$21: track 69.8 -> 110.6 mm, vias 3 -> 1
- net OXO: track 206.8 -> 246.1 mm, vias 4 -> 7
- net 3V3: track 311.0 -> 346.5 mm, vias 7 -> 4
- net XOO: track 234.9 -> 204.5 mm, vias 5 -> 6
- net N$30: track 82.2 -> 112.2 mm
- net N$9: track 154.5 -> 180.3 mm, vias 4 -> 3
- net OOX: track 238.5 -> 213.2 mm
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